Commit message: finish mapping and navigation

File: keigan_motor_description/urdf/keigan_motor.urdf.xacro (robot description, xacro)
@@ -17,5 +17,5 @@
   <link name="laser"/>
   <joint name="laser_joint" type="fixed">
-    <origin xyz="-1.3 0 0.4938" rpy="0 0 ${M_PI}" />
+    <origin xyz="-0.013 0 0.3938" rpy="0 0 ${M_PI}" />
     <parent link="base_link" />
     <child link="laser" />
